File: BufferedMult.kicad_pcb (KiCad board)
At the start: 2 copper layers, 20 x 108 mm, 27 parts, among them J1 EURORACK_PWR_10PIN, J2 IN_1, J3 OUT_1A, J4 OUT_1B, J5 OUT_1C, J6 IN_2, J7 OUT_2A, J8 OUT_2B, J9 OUT_2C, U1 TL074, U2 TL074

Commit message: Update PCB
Parts:
- C1, C2: footprint Capacitor_SMD:CP_Elec_6.3x5.4 -> Capacitor_THT:CP_Radial_D5.0mm_P2.00mm; moved to F.Cu
- J1: footprint Connector_IDC:IDC-Header_2x05_P2.54mm_Vertical_SMD -> Connector_IDC:IDC-Header_2x05_P2.54mm_Vertical
- moved R7 91.1 mm to (24.9, 99.9), turned to -90 degrees
- moved R3 90.7 mm to (25.0, 54.6), turned to -90 degrees
- moved U1 85.5 mm to (30.0, 26.2)
- moved R1 85.2 mm to (36.9, 22.0), turned to 0 degrees
- moved C4 84.1 mm to (23.4, 26.5), turned to 0 degrees
- moved R2 82.4 mm to (35.0, 40.1), turned to -90 degrees
- moved U2 81.3 mm to (30.0, 69.0)
- moved C6 81.3 mm to (22.9, 68.0), turned to -90 degrees
- moved R4 81.0 mm to (35.0, 54.6), turned to -90 degrees
- moved R8 80.7 mm to (35.0, 99.6), turned to -90 degrees
- moved R5 80.5 mm to (36.9, 66.4), turned to 90 degrees
- moved R6 80.5 mm to (35.0, 85.4), turned to -90 degrees
- moved C3 72.8 mm to (37.0, 26.5), turned to 0 degrees
- moved C5 67.8 mm to (37.0, 70.0), turned to -90 degrees
- moved C2 51.6 mm to (24.5, 123.5), turned to -90 degrees
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- renumbered C4 to C3, C3 to C4, C6 to C5, C5 to C6, D2 to D1, D1 to D2
Connections:
- C3 pad 1: GND -> +12V
- C3 pad 2: -12V -> GND
- C4 pad 1: +12V -> GND
- C4 pad 2: GND -> -12V
- C5 pad 1: GND -> +12V
- C5 pad 2: -12V -> GND
- C6 pad 1: +12V -> GND
- C6 pad 2: GND -> -12V
- D1 pad 1: -12V_RAW -> +12V
- D1 pad 2: -12V -> +12V_RAW
- D2 pad 1: +12V -> -12V_RAW
- D2 pad 2: +12V_RAW -> -12V

Commit message: Reposition parts and flood the ground planes
Parts:
- moved R5 50.5 mm to (36.9, 117.0)
- moved U2 50.5 mm to (30.0, 119.5)
- moved C5 50.5 mm to (37.0, 120.5)
- moved C6 50.5 mm to (23.0, 118.5)
- moved C1 44.5 mm to (24.5, 64.0)
- moved C2 44.5 mm to (24.5, 79.0)
- moved D1 44.5 mm to (24.5, 70.4)
- moved D2 44.5 mm to (24.5, 75.0)
- moved J1 44.5 mm to (33.5, 77.1)
- moved R6 8.10 mm to (35.0, 93.5)
- moved R7 8.10 mm to (24.9, 108.0)
- moved J6 8.10 mm to (25.0, 85.6)
- moved J7 8.10 mm to (35.0, 85.6)
- moved J8 8.10 mm to (25.0, 100.1)
- moved J9 8.10 mm to (35.0, 100.1)
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Routing:
- added copper zone on B.Cu, net (none)
- added copper zone on F.Cu, net (none)

Commit message: Repositioning components
Parts:
- moved C2 1.04 mm to (24.5, 80.0)
- moved C1 0.50 mm to (24.5, 63.5)
- moved U2 0.50 mm to (30.0, 120.0)
- moved R2 0.41 mm to (35.0, 40.5)
- moved R3 0.41 mm to (25.0, 55.0)
- moved R4 0.41 mm to (35.0, 55.0)
- moved R8 0.31 mm to (35.0, 108.0)
- moved U1 0.19 mm to (30.0, 26.0)
- moved J6 0.10 mm to (25.0, 85.5)
- moved J7 0.10 mm to (35.0, 85.5)
- moved J8 0.10 mm to (25.0, 100.0)
- moved J9 0.10 mm to (35.0, 100.0)
- moved D1 0.09 mm to (24.5, 70.5)
- moved R7 0.09 mm to (25.0, 108.0)
Routing:
- added copper zone on B.Cu, net GND
- added copper zone on F.Cu, net GND
- removed copper zone on B.Cu, net (none)
- removed copper zone on F.Cu, net (none)

Commit message: Update BufferedMult.kicad_pcb
Routing:
- net +12V: track 0.00 -> 130.0 mm, vias 0 -> 2
- net -12V: track 0.00 -> 117.2 mm, vias 0 -> 2
- net CH1_BUF: track 0.00 -> 80.5 mm, vias 0 -> 1
- net CH1_OP_C: track 0.00 -> 48.0 mm
- net CH2_OP_A: track 0.00 -> 40.2 mm
- net CH1_IN: track 0.00 -> 38.3 mm
- net CH2_IN: track 0.00 -> 32.9 mm
- net CH1_OP_B: track 0.00 -> 29.5 mm
- net CH2_OP_B: track 0.00 -> 24.9 mm
- net CH2_BUF: track 0.00 -> 14.9 mm
- net CH2_OP_C: track 0.00 -> 13.5 mm
- net CH1_OP_A: track 0.00 -> 12.2 mm
- net +12V_RAW: track 0.00 -> 11.0 mm
- net -12V_RAW: track 0.00 -> 10.4 mm
- net CH2_OUT_C: track 0.00 -> 2.49 mm
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Other:
- board text added: "-12V"
- board text added: "github.com/domesticmouse/BufferedMult-SKiDL"

Commit message: Re-route
Routing:
- net CH1_BUF: track 80.5 -> 83.8 mm
- net GND: vias 8 -> 12
Other:
- board text added: "Version: 1.1"

Commit message: Switch quad op-amps U1/U2 from TL074CDR to TL074HIDR (LCSC C2878713)
- Update `buffered_multiple.py` op-amp value (`TL074H`), MPN (`TL074HIDR`), and LCSC part number (`C2878713`).
- Regenerate KiCad netlist, XML BOM, JLCPCB SMT BOM CSV, and hierarchical schematic SVGs.
- Update `U1` and `U2` footprint properties in `BufferedMult.kicad_pcb` and `production/bom.csv`.
- Update BOM tables and signal flow documentation in `README.md` and `PCB_LAYOUT_GUIDE.md`.
Parts:
- U1, U2: value TL074 -> TL074H
Changed lines of the file:
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@@
 			)
 		)
-		(property "Value" "TL074"
+		(property "Value" "TL074H"
 			(at 0 -5.28 0)
 			(layer "B.SilkS")
@@
 			)
 		)
-		(property "LCSC" "C12594"
-			(at 0 0 0)
-			(unlocked yes)
-			(layer "B.Fab")
-			(hide yes)
-			(effects
-				(font
-					(size 1 1)
-					(thickness 0.15)
-				)
-				(justify mirror)
-			)
-		)
-		(property "MPN" "TL074CDR"
+		(property "LCSC" "C2878713"
+			(at 0 0 0)
+			(unlocked yes)
+			(layer "B.Fab")
+			(hide yes)
+			(effects
+				(font
+					(size 1 1)
+					(thickness 0.15)
+				)
+				(justify mirror)
+			)
+		)
+		(property "MPN" "TL074HIDR"
 			(at 0 0 0)
 			(unlocked yes)
@@
 			)
 		)
-		(property "Value" "TL074"
+		(property "Value" "TL074H"
 			(at 0 -5.28 0)
 			(layer "B.SilkS")
@@
 			)
 		)
-		(property "LCSC" "C12594"
-			(at 0 0 0)
-			(unlocked yes)
-			(layer "B.Fab")
-			(hide yes)
-			(effects
-				(font
-					(size 1 1)
-					(thickness 0.15)
-				)
-				(justify mirror)
-			)
-		)
-		(property "MPN" "TL074CDR"
-			(at 0 0 0)
-			(unlocked yes)
+		(property "LCSC" "C2878713"
+			(at 0 0 0)
+			(unlocked yes)
+			(layer "B.Fab")
+			(hide yes)
+			(effects
+				(font
+					(size 1 1)
+					(thickness 0.15)
+				)
+				(justify mirror)
+			)
+		)
+		(property "MPN" "TL074HIDR"
+			(at 0 0 0)
+			(unlocked yes)
