File: BufferedMult.kicad_pcb (KiCad board)
At the start: 2 copper layers, 20 x 108 mm, 27 parts, among them J1 EURORACK_PWR_10PIN, J2 IN_1, J3 OUT_1A, J4 OUT_1B, J5 OUT_1C, J6 IN_2, J7 OUT_2A, J8 OUT_2B, J9 OUT_2C, U1 TL074H, U2 TL074H

Commit message: Re-route power lines
Routing:
- net -12V: track 117.5 -> 118.2 mm
- net CH1_IN: track 38.3 -> 37.8 mm
Changed lines of the file:
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@@
-	)
-	(segment
-		(start 32.642107 119.832893)
-		(end 32.475 120)
-		(width 0.5)
-		(layer "B.Cu")
-		(net "+12V")
 	)
 	(segment
@@
 	)
 	(segment
+		(start 34.5 119.54)
+		(end 34.332893 119.707107)
+		(width 0.5)
+		(layer "B.Cu")
+		(net "+12V")
+	)
+	(segment
 		(start 36.975 119.54)
 		(end 34.5 119.54)
@@
 	)
 	(segment
-		(start 34.5 119.54)
-		(end 33.349214 119.54)
-		(width 0.5)
-		(layer "B.Cu")
-		(net "+12V")
-	)
-	(segment
 		(start 22.5 70.5)
 		(end 21.792893 69.792893)
@@
 		(start 21.5 69.085786)
 		(end 21.5 64.5)
+		(width 0.5)
+		(layer "B.Cu")
+		(net "+12V")
+	)
+	(segment
+		(start 33.625786 120)
+		(end 32.475 120)
 		(width 0.5)
 		(layer "B.Cu")
@@
 	)
 	(arc
-		(start 33.349214 119.54)
-		(mid 32.966531 119.61612)
-		(end 32.642107 119.832893)
+		(start 33.625786 120)
+		(mid 34.008469 119.92388)
+		(end 34.332893 119.707107)
 		(width 0.5)
 		(layer "B.Cu")
@@
 	)
 	(segment
+		(start 31.2 37.7)
+		(end 31.2 28.189448)
+		(width 0.2)
+		(layer "B.Cu")
+		(net "CH1_IN")
+	)
+	(segment
+		(start 33.915256 28.915256)
+		(end 35.5 30.5)
+		(width 0.2)
+		(layer "B.Cu")
+		(net "CH1_IN")
+	)
+	(segment
+		(start 38.4 30.1)
+		(end 38.4 26.3125)
+		(width 0.2)
+		(layer "B.Cu")
+		(net "CH1_IN")
+	)
+	(segment
+		(start 38.4 26.3125)
+		(end 36.9125 24.825)
+		(width 0.2)
+		(layer "B.Cu")
+		(net "CH1_IN")
+	)
+	(segment
+		(start 36.9125 24.825)
+		(end 32.57 24.825)
+		(width 0.2)
+		(layer "B.Cu")
+		(net "CH1_IN")
+	)
+	(segment
 		(start 31.2 28.189448)
 		(end 31.474192 27.915256)
@@
 	)
 	(segment
-		(start 31.2 37.7)
-		(end 31.2 28.189448)
+		(start 25 43.9)
+		(end 31.2 37.7)
+		(width 0.2)
+		(layer "B.Cu")
+		(net "CH1_IN")
+	)
+	(segment
+		(start 35.5 30.5)
+		(end 38 30.5)
+		(width 0.2)
+		(layer "B.Cu")
+		(net "CH1_IN")
+	)
+	(segment
+		(start 31.474192 27.915256)
+		(end 33.915256 27.915256)
+		(width 0.2)
+		(layer "B.Cu")
+		(net "CH1_IN")
+	)
+	(segment
+		(start 32.57 24.825)
+		(end 32.475 24.73)
 		(width 0.2)
 		(layer "B.Cu")
@@
 	)
 	(segment
-		(start 31.474192 27.915256)
-		(end 33.915256 27.915256)
-		(width 0.2)
-		(layer "B.Cu")
-		(net "CH1_IN")
-	)
-	(segment
-		(start 38.6 26.5125)
-		(end 36.9125 24.825)
-		(width 0.2)
-		(layer "B.Cu")
-		(net "CH1_IN")
-	)
-	(segment
-		(start 36.9125 24.825)
-		(end 32.57 24.825)
-		(width 0.2)
-		(layer "B.Cu")
-		(net "CH1_IN")
-	)
-	(segment
-		(start 33.915256 28.915256)
-		(end 35.5 30.5)
-		(width 0.2)
-		(layer "B.Cu")
-		(net "CH1_IN")
-	)
-	(segment
-		(start 38.6 30.5)
-		(end 38.6 26.5125)
-		(width 0.2)
-		(layer "B.Cu")
-		(net "CH1_IN")
-	)
-	(segment
-		(start 32.57 24.825)
-		(end 32.475 24.73)
-		(width 0.2)
-		(layer "B.Cu")
-		(net "CH1_IN")
-	)
-	(segment
-		(start 25 43.9)
-		(end 31.2 37.7)
-		(width 0.2)
-		(layer "B.Cu")
-		(net "CH1_IN")
-	)
-	(segment
-		(start 35.5 30.5)
-		(end 38.6 30.5)
+		(start 38 30.5)
+		(end 38.4 30.1)
 		(width 0.2)
 		(layer "B.Cu")
@@
 	)
 	(segment
+		(start 22.5 75)
+		(end 22.5 81)
+		(width 0.5)
+		(layer "B.Cu")
+		(net "-12V")
+	)
+	(segment
 		(start 22.975 119.44)
 		(end 25.5 119.44)
@@
 	)
 	(segment
-		(start 22.5 79)
-		(end 22.5 79.585786)
-		(width 0.5)
-		(layer "B.Cu")
-		(net "-12V")
-	)
-	(segment
 		(start 23.45 27.45)
 		(end 24.9 26)
@@
 	)
 	(segment
-		(start 27.257893 119.732893)
+		(start 23.5 82)
+		(end 24.5 82)
+		(width 0.5)
+		(layer "B.Cu")
+		(net "-12V")
+	)
+	(segment
+		(start 26.514214 120)
 		(end 27.525 120)
 		(width 0.5)
@@
 	(segment
 		(start 25.5 119.44)
-		(end 26.550786 119.44)
-		(width 0.5)
-		(layer "B.Cu")
-		(net "-12V")
-	)
-	(segment
-		(start 22.5 75)
-		(end 22.5 79)
+		(end 25.54 119.44)
+		(width 0.5)
+		(layer "B.Cu")
+		(net "-12V")
+	)
+	(segment
+		(start 25.54 119.44)
+		(end 25.807107 119.707107)
 		(width 0.5)
 		(layer "B.Cu")
@@
 		(net "-12V")
 	)
-	(segment
-		(start 22.792893 80.292893)
-		(end 24.5 82)
-		(width 0.5)
-		(layer "B.Cu")
-		(net "-12V")
-	)
-	(arc
-		(start 22.792893 80.292893)
-		(mid 22.57612 79.96847)
-		(end 22.5 79.585786)
-		(width 0.5)
-		(layer "B.Cu")
-		(net "-12V")
-	)
-	(arc
-		(start 26.550786 119.44)
-		(mid 26.933469 119.51612)
-		(end 27.257893 119.732893)
-		(width 0.5)
-		(layer "B.Cu")
+	(arc
+		(start 23.5 82)
+		(mid 22.792893 81.707107)
+		(end 22.5 81)
+		(width 0.5)
+		(layer "B.Cu")
+		(net "-12V")
+	)
+	(arc
+		(start 26.514214 120)
+		(mid 26.131531 119.92388)
+		(end 25.807107 119.707107)
+		(width 0.5)
+		(layer "B.Cu")
