File: BufferedMult_Panel.kicad_pcb (KiCad board)
At the start: 2 copper layers, 20 x 128.5 mm, 10 parts, among them J2 IN_1, J3 OUT_1A, J4 OUT_1B, J5 OUT_1C, J6 IN_2, J7 OUT_2A, J8 OUT_2B, J9 OUT_2C

Commit message: Add `eurorack-panel` skill and update 4HP front panel PCB and Gerbers
- Package the front panel generator into `.agents/skills/eurorack-panel/` with `SKILL.md`, `scripts/generate_eurorack_panel.py`, and `references/eurorack_mechanical_spec.md`
- Remove standalone root `generate_panel.py` and document the skill CLI workflow in `FRONT_PANEL_GUIDE.md`
- Update `BufferedMult_Panel` KiCad project files and regenerate fabrication Gerbers and Excellon drill outputs in `production/`
Other:
- board text removed: "1 -> 2"
- board text removed: "1:3 / 1:6"
- board text removed: "JLCJLCJLCJLC"
- board text removed: "NORM"
Changed lines of the file:
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@@
 	)
 	(gr_line
-		(start 22 22.75)
-		(end 38 22.75)
+		(start 22 25.75)
+		(end 38 25.75)
 		(stroke
 			(width 0.25)
@@
 		(layer "F.SilkS")
 	)
-	(gr_line
-		(start 23.9 80.2)
-		(end 25 81.7)
+	(gr_rect
+		(start 26 120)
+		(end 34 128)
 		(stroke
-			(width 0.25)
+			(width 0.1)
 			(type solid)
 		)
-		(layer "F.SilkS")
-	)
-	(gr_line
-		(start 25 63.8)
-		(end 25 81.5)
-		(stroke
-			(width 0.25)
-			(type dash)
-		)
-		(layer "F.SilkS")
-	)
-	(gr_line
-		(start 26.1 80.2)
-		(end 25 81.7)
-		(stroke
-			(width 0.25)
-			(type solid)
-		)
-		(layer "F.SilkS")
+		(fill yes)
+		(layer "B.SilkS")
 	)
 	(gr_rect
@@
 		(fill no)
 		(layer "B.Fab")
-	)
-	(gr_text "NORM"
-		(at 33.5 71.55 0)
-		(layer "F.SilkS")
-		(effects
-			(font
-				(size 1.1 1.1)
-				(thickness 0.18)
-			)
-		)
-	)
-	(gr_text "1 -> 2"
-		(at 33.5 73.95 0)
-		(layer "F.SilkS")
-		(effects
-			(font
-				(size 1.1 1.1)
-				(thickness 0.18)
-			)
-		)
 	)
 	(gr_text "OUT 1B"
@@
 		)
 	)
-	(gr_text "1:3 / 1:6"
-		(at 30 122.25 0)
-		(layer "F.SilkS")
-		(effects
-			(font
-				(size 1.3 1.3)
-				(thickness 0.22)
-				(bold yes)
-			)
-		)
-	)
 	(gr_text "BUF MULT"
-		(at 30 20 0)
+		(at 30 23 0)
 		(layer "F.SilkS")
 		(effects
@@
 		(layer "B.SilkS")
 		(effects
-			(font
-				(size 1 1)
-				(thickness 0.15)
-			)
-			(justify mirror)
-		)
-	)
-	(gr_text "JLCJLCJLCJLC"
-		(at 30 72.73 0)
-		(layer "B.SilkS")
-		(effects
